File: hardware/keyboard_simple.kicad_pcb (KiCad board)
At the start: 2 copper layers, 228.6 x 76.2 mm, 60 parts, among them U1 74HC165, U2 74HC165, U3 74HC165, U4 74HC165, U5 XW06A, U6 74HC165, U7 74HC165

Commit message: layout doing
Parts:
- added C1: 100nF, Capacitor_SMD:C_0603_1608Metric, F.Cu at (190.9, 112.7)
- added C10: 104, Capacitor_SMD:C_0603_1608Metric, B.Cu at (212.7, 96.0)
- added C11: 104, Capacitor_SMD:C_0603_1608Metric, B.Cu at (211.0, 96.0)
- added C12: 10uF, Capacitor_SMD:C_1206_3216Metric, F.Cu at (135.5, 105.4)
- added C13: 22pF, Capacitor_SMD:C_0603_1608Metric, B.Cu at (227.2, 99.8)
- added C14: 1uF, Capacitor_SMD:C_0603_1608Metric, F.Cu at (142.4, 105.6)
- added C15: 22pF, Capacitor_SMD:C_0603_1608Metric, B.Cu at (227.2, 102.8)
- added C2: 0.1uF, Capacitor_SMD:C_0603_1608Metric, F.Cu at (202.8, 99.8)
- added C3: 0.1uF, Capacitor_SMD:C_0603_1608Metric, F.Cu at (189.4, 97.0)
- added C4: 0.1uF, Capacitor_SMD:C_0603_1608Metric, F.Cu at (187.4, 99.3)
- added C5: 0.1uF, Capacitor_SMD:C_0603_1608Metric, F.Cu at (185.6, 105.9)
- added C6: 0.1uF, Capacitor_SMD:C_0603_1608Metric, F.Cu at (200.8, 112.5)
- added C7: 0.1uF, Capacitor_SMD:C_0603_1608Metric, B.Cu at (154.3, 100.3)
- added C8: 22pF, Capacitor_SMD:C_0603_1608Metric, F.Cu at (178.5, 102.1)
- added C9: 22pF, Capacitor_SMD:C_0603_1608Metric, F.Cu at (181.8, 102.1)
- added D1: LED, LED_SMD:LED_0805_2012Metric, B.Cu at (144.2, 110.2)
- added D3: LED, LED_SMD:LED_0805_2012Metric, B.Cu at (268.4, 73.4)
- added D5: 1N4148W, Diode_SMD:D_SOD-123, B.Cu at (216.8, 110.7)
- added J1: USB_C_Receptacle_USB2.0, EnergyVortex:USB_C_Receptacle_HRO_TYPE-C-31-M-12, B.Cu at (151.5, 113.5)
- added J2: Conn_02x09_Odd_Even, Connector_PinHeader_2.54mm:PinHeader_2x09_P2.54mm_Vertical_SMD, B.Cu at (252.9, 93.2)
- added J3: Conn_02x09_Odd_Even, Connector_PinHeader_2.54mm:PinHeader_2x09_P2.54mm_Vertical_SMD, B.Cu at (250.8, 111.2)
- added J4: USB_C_Receptacle_USB2.0, EnergyVortex:USB_C_Receptacle_HRO_TYPE-C-31-M-12, B.Cu at (271.2, 63.2)
- added J5: Conn_01x04, Connector_PinHeader_2.54mm:PinHeader_1x04_P2.54mm_Vertical, F.Cu at (209.9, 102.3)
- added J6: Conn_02x04_Odd_Even, Connector_PinHeader_2.54mm:PinHeader_2x04_P2.54mm_Vertical, F.Cu at (176.4, 113.3)
- added JP1: SolderJumper_2_Open, Jumper:SolderJumper-2_P1.3mm_Open_TrianglePad1.0x1.5mm, B.Cu at (138.3, 112.2)
- added JP2: SolderJumper_2_Open, Jumper:SolderJumper-2_P1.3mm_Open_TrianglePad1.0x1.5mm, B.Cu at (271.7, 73.4)
- added LED1: WS2812B-2020, EnergyVortex:LED_WS2812B-B, F.Cu at (54.5, 52.8)
- added LED10: WS2812B-2020, EnergyVortex:LED_WS2812B-B, F.Cu at (226.2, 52.8)
- added LED11: WS2812B-2020, EnergyVortex:LED_WS2812B-B, F.Cu at (245.3, 52.8)
- added LED12: WS2812B-2020, EnergyVortex:LED_WS2812B-B, F.Cu at (264.3, 52.8)
- added LED13: WS2812B-2020, EnergyVortex:LED_WS2812B-B, F.Cu at (257.2, 71.9)
- added LED14: WS2812B-2020, EnergyVortex:LED_WS2812B-B, F.Cu at (231.0, 71.9)
- added LED15: WS2812B-2020, EnergyVortex:LED_WS2812B-B, F.Cu at (212.0, 71.9)
- added LED16: WS2812B-2020, EnergyVortex:LED_WS2812B-B, F.Cu at (192.9, 71.9)
- added LED17: WS2812B-2020, EnergyVortex:LED_WS2812B-B, F.Cu at (173.8, 71.9)
- added LED18: WS2812B-2020, EnergyVortex:LED_WS2812B-B, F.Cu at (154.8, 71.9)
- added LED19: WS2812B-2020, EnergyVortex:LED_WS2812B-B, F.Cu at (57.0, 71.9)
- added LED2: WS2812B-2020, EnergyVortex:LED_WS2812B-B, F.Cu at (72.8, 52.8)
- added LED20: WS2812B-2020, EnergyVortex:LED_WS2812B-B, F.Cu at (78.6, 71.9)
- added LED21: WS2812B-2020, EnergyVortex:LED_WS2812B-B, F.Cu at (97.6, 71.9)
- added LED22: WS2812B-2020, EnergyVortex:LED_WS2812B-B, F.Cu at (116.7, 71.9)
- added LED23: WS2812B-2020, EnergyVortex:LED_WS2812B-B, F.Cu at (135.8, 71.9)
- added LED24: WS2812B-2020, EnergyVortex:LED_WS2812B-B, F.Cu at (262.0, 90.9)
- added LED25: WS2812B-2020, EnergyVortex:LED_WS2812B-B, F.Cu at (240.4, 90.9)
- added LED26: WS2812B-2020, EnergyVortex:LED_WS2812B-B, F.Cu at (221.4, 90.9)
- added LED27: WS2812B-2020, EnergyVortex:LED_WS2812B-B, F.Cu at (202.3, 90.9)
- added LED28: WS2812B-2020, EnergyVortex:LED_WS2812B-B, F.Cu at (183.4, 90.9)
- added LED29: WS2812B-2020, EnergyVortex:LED_WS2812B-B, F.Cu at (164.2, 90.9)
- added LED3: WS2812B-2020, EnergyVortex:LED_WS2812B-B, F.Cu at (90.6, 52.8)
- added LED30: WS2812B-2020, EnergyVortex:LED_WS2812B-B, F.Cu at (145.4, 90.9)
- added LED31: WS2812B-2020, EnergyVortex:LED_WS2812B-B, F.Cu at (126.3, 90.9)
- added LED32: WS2812B-2020, EnergyVortex:LED_WS2812B-B, F.Cu at (107.2, 90.9)
- added LED33: WS2812B-2020, EnergyVortex:LED_WS2812B-B, F.Cu at (88.1, 90.9)
- added LED34: WS2812B-2020, EnergyVortex:LED_WS2812B-B, F.Cu at (61.9, 90.9)
- added LED35: WS2812B-2020, EnergyVortex:LED_WS2812B-B, F.Cu at (57.1, 110.0)
- added LED36: WS2812B-2020, EnergyVortex:LED_WS2812B-B, F.Cu at (78.6, 110.0)
- added LED37: WS2812B-2020, EnergyVortex:LED_WS2812B-B, F.Cu at (97.7, 110.0)
- added LED38: WS2812B-2020, EnergyVortex:LED_WS2812B-B, F.Cu at (166.8, 110.0)
- added LED39: WS2812B-2020, EnergyVortex:LED_WS2812B-B, F.Cu at (238.1, 110.0)
- added LED4: WS2812B-2020, EnergyVortex:LED_WS2812B-B, F.Cu at (111.9, 52.8)
- added LED40: WS2812B-2020, EnergyVortex:LED_WS2812B-B, F.Cu at (262.0, 110.0)
- added LED5: WS2812B-2020, EnergyVortex:LED_WS2812B-B, F.Cu at (130.9, 52.8)
- added LED6: WS2812B-2020, EnergyVortex:LED_WS2812B-B, F.Cu at (149.9, 52.8)
- added LED7: WS2812B-2020, EnergyVortex:LED_WS2812B-B, F.Cu at (169.1, 52.8)
- added LED8: WS2812B-2020, EnergyVortex:LED_WS2812B-B, F.Cu at (188.1, 52.8)
- added LED9: WS2812B-2020, EnergyVortex:LED_WS2812B-B, F.Cu at (207.2, 52.8)
- added Q1: S8050, Package_TO_SOT_SMD:SOT-23, B.Cu at (221.9, 108.2)
- added Q2: S8550, Package_TO_SOT_SMD:SOT-23, B.Cu at (225.9, 112.5)
- added R1: 10k, Resistor_SMD:R_0603_1608Metric, B.Cu at (142.1, 113.5)
- added R10: 10K, Resistor_SMD:R_0603_1608Metric, F.Cu at (206.9, 99.8)
- added R11: 1k, Resistor_SMD:R_0603_1608Metric, B.Cu at (217.8, 107.9)
- added R12: 1k, Resistor_SMD:R_0603_1608Metric, B.Cu at (226.2, 109.2)
- added R13: 1k, Resistor_SMD:R_0603_1608Metric, B.Cu at (226.2, 107.2)
- added R15: 2k, Resistor_SMD:R_0603_1608Metric, B.Cu at (221.9, 112.2)
- added R2: 2k, Resistor_SMD:R_0603_1608Metric, B.Cu at (148.0, 106.6)
- added R3: 10K, Resistor_SMD:R_0603_1608Metric, B.Cu at (154.3, 97.3)
- added R4: 10k, Resistor_SMD:R_0603_1608Metric, B.Cu at (263.5, 57.6)
- added R5: 2k, Resistor_SMD:R_0603_1608Metric, B.Cu at (269.1, 69.8)
- added R6: 22, Resistor_SMD:R_0603_1608Metric, B.Cu at (265.8, 73.4)
- added R7: 22, Resistor_SMD:R_0603_1608Metric, B.Cu at (263.8, 73.4)
- added R8: 1.5K, Resistor_SMD:R_0603_1608Metric, B.Cu at (265.6, 69.8)
- added R9: 10K, Resistor_SMD:R_0603_1608Metric, F.Cu at (204.9, 99.8)
- added SW1: SW_Push, EnergyVortex:SW_Push_1P1T_NO_6x6mm_H9.5mm, B.Cu at (146.7, 98.5)
- added U5: STM32F103RBTx, Package_QFP:LQFP-64_10x10mm_P0.5mm, F.Cu at (194.7, 104.6)
- added U8: XC6210B332MR, Package_TO_SOT_SMD:SOT-23-5, F.Cu at (139.3, 105.1)
- added U9: CH340G, Package_SO:SOIC-16_3.9x9.9mm_P1.27mm, B.Cu at (217.8, 99.5)
- added Y1: 8M, EnergyVortex:Crystal_SMD_Qantek_QC5CB-2Pin_5x3.2mm, F.Cu at (180.0, 99.0)
- added Y2: 12M, EnergyVortex:Crystal_SMD_Qantek_QC5CB-2Pin_5x3.2mm, B.Cu at (224.4, 101.3)
- RN1: renamed from RN4; moved to B.Cu
- RN3: renamed from RN2; moved to B.Cu
- RN4: renamed from RN3; moved to B.Cu
- S1: renamed from S25; footprint EnergyVortex:CHERRY-MX-LED -> EnergyVortex:CHERRY-MX-LED+
- S10: renamed from S2; footprint EnergyVortex:CHERRY-MX-LED -> EnergyVortex:CHERRY-MX-LED+
- S11: renamed from S3; footprint EnergyVortex:CHERRY-MX-LED -> EnergyVortex:CHERRY-MX-LED+
- S12: renamed from S4; footprint EnergyVortex:CHERRY-MX-LED -> EnergyVortex:CHERRY-MX-LED+
- S13: renamed from S5; footprint EnergyVortex:CHERRY-MX-LED -> EnergyVortex:CHERRY-MX-LED+
- S14: renamed from S6; footprint EnergyVortex:CHERRY-MX-LED -> EnergyVortex:CHERRY-MX-LED+
- S15: renamed from S7; footprint EnergyVortex:CHERRY-MX-LED -> EnergyVortex:CHERRY-MX-LED+
- S16: renamed from S8; footprint EnergyVortex:CHERRY-MX-LED -> EnergyVortex:CHERRY-MX-LED+
- S17: renamed from S9; footprint EnergyVortex:CHERRY-MX-LED -> EnergyVortex:CHERRY-MX-LED+
- S18: renamed from S10; footprint EnergyVortex:CHERRY-MX-LED -> EnergyVortex:CHERRY-MX-LED+
- S19: renamed from S11; footprint EnergyVortex:CHERRY-MX-LED -> EnergyVortex:CHERRY-MX-LED+
- S2: renamed from S26; footprint EnergyVortex:CHERRY-MX-LED -> EnergyVortex:CHERRY-MX-LED+
- S20: renamed from S12; footprint EnergyVortex:CHERRY-MX-LED -> EnergyVortex:CHERRY-MX-LED+
- S21: renamed from S13; footprint EnergyVortex:CHERRY-MX-LED -> EnergyVortex:CHERRY-MX-LED+
- S22: renamed from S14; footprint EnergyVortex:CHERRY-MX-LED -> EnergyVortex:CHERRY-MX-LED+
- S23: renamed from S15; footprint EnergyVortex:CHERRY-MX-LED -> EnergyVortex:CHERRY-MX-LED+
- S24: renamed from S16; footprint EnergyVortex:CHERRY-MX-LED -> EnergyVortex:CHERRY-MX-LED+
- S25: renamed from S17; footprint EnergyVortex:CHERRY-MX-LED -> EnergyVortex:CHERRY-MX-LED+
- S26: renamed from S18; footprint EnergyVortex:CHERRY-MX-LED -> EnergyVortex:CHERRY-MX-LED+
- S27: renamed from S19; footprint EnergyVortex:CHERRY-MX-LED -> EnergyVortex:CHERRY-MX-LED+
- S28: renamed from S20; footprint EnergyVortex:CHERRY-MX-LED -> EnergyVortex:CHERRY-MX-LED+
- S29: renamed from S21; footprint EnergyVortex:CHERRY-MX-LED -> EnergyVortex:CHERRY-MX-LED+
- S3: renamed from S27; footprint EnergyVortex:CHERRY-MX-LED -> EnergyVortex:CHERRY-MX-LED+
- S30: renamed from S22; footprint EnergyVortex:CHERRY-MX-LED -> EnergyVortex:CHERRY-MX-LED+
- S31: renamed from S23; footprint EnergyVortex:CHERRY-MX-LED -> EnergyVortex:CHERRY-MX-LED+
- S32: renamed from S24; footprint EnergyVortex:CHERRY-MX-LED -> EnergyVortex:CHERRY-MX-LED+
- S33: renamed from S35; footprint EnergyVortex:CHERRY-MX-LED -> EnergyVortex:CHERRY-MX-LED+
- S34: renamed from S36; footprint EnergyVortex:CHERRY-MX-LED -> EnergyVortex:CHERRY-MX-LED+
- S35: renamed from S37; footprint EnergyVortex:CHERRY-MX-LED -> EnergyVortex:CHERRY-MX-LED+
- S36: renamed from S38; footprint EnergyVortex:CHERRY-MX-LED -> EnergyVortex:CHERRY-MX-LED+
- S37: renamed from S39; footprint EnergyVortex:CHERRY-MX-LED -> EnergyVortex:CHERRY-MX-LED+
- S38: renamed from S40; footprint EnergyVortex:CHERRY-MX-LED -> EnergyVortex:CHERRY-MX-LED+
- S39: renamed from S33; footprint EnergyVortex:CHERRY-MX-LED -> EnergyVortex:CHERRY-MX-LED+
- S4: renamed from S28; footprint EnergyVortex:CHERRY-MX-LED -> EnergyVortex:CHERRY-MX-LED+
- S40: renamed from S34; footprint EnergyVortex:CHERRY-MX-LED -> EnergyVortex:CHERRY-MX-LED+
- S5: renamed from S29; footprint EnergyVortex:CHERRY-MX-LED -> EnergyVortex:CHERRY-MX-LED+
- S6: renamed from S30; footprint EnergyVortex:CHERRY-MX-LED -> EnergyVortex:CHERRY-MX-LED+
- S7: renamed from S31; footprint EnergyVortex:CHERRY-MX-LED -> EnergyVortex:CHERRY-MX-LED+
- S8: renamed from S32; footprint EnergyVortex:CHERRY-MX-LED -> EnergyVortex:CHERRY-MX-LED+
- S9: renamed from S1; footprint EnergyVortex:CHERRY-MX-LED -> EnergyVortex:CHERRY-MX-LED+
- U2, U3, U4: moved to B.Cu
- moved RN5 244.9 mm to (244.2, 58.1), turned to 90 degrees
- moved U6 193.8 mm to (243.7, 67.3)
- moved RN1 193.5 mm to (197.8, 49.2), turned to 90 degrees
- moved U4 157.9 mm to (197.2, 54.8), turned to -90 degrees
- moved RN6 155.3 mm to (111.6, 110.7), turned to -90 degrees
- moved U10 151.5 mm to (123.8, 99.8), turned to 180 degrees
- moved R17 148.5 mm to (130.4, 95.5), turned to 180 degrees
- moved R14 147.5 mm to (121.9, 111.7)
- moved C16 147.5 mm to (129.9, 106.7)
- moved C17 147.5 mm to (121.9, 109.2)
- moved C18 147.5 mm to (125.9, 109.2)
- moved R16 146.0 mm to (130.4, 97.3), turned to 180 degrees
- moved RN4 144.0 mm to (145.4, 68.0), turned to 90 degrees
- moved RN7 143.2 mm to (130.4, 100.3)
- moved U7 125.9 mm to (111.9, 102.3)
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- renumbered C3 to C16, C2 to C17, C1 to C18, R3 to R14, R1 to R16, R2 to R17, RN1 to RN2, RN7 to RN5, RN5 to RN7, U5 to U10, U7 to U6, U6 to U7
