File: hardware/keyboard_simple.kicad_sch (KiCad schematic)
At the start: 129 parts, among them J1 FPC, U1 74HC165, U2 74HC165, U3 74HC165, U4 74HC165, U5 XW06A, U6 74HC165, U7 74HC165

Commit message: layout doing
Parts:
- removed D? (x2): 1N4007, Diode_SMD:D_SOD-123F, symbol Device:D
- removed J?: Conn_02x18_Odd_Even, Connector_PinHeader_2.54mm:PinHeader_2x18_P2.54mm_Vertical, symbol Connector_Generic:Conn_02x18_Odd_Even
- removed J?: Conn_01x03, symbol Connector_Generic:Conn_01x03
- added J2, J3: Conn_02x09_Odd_Even, Connector_PinHeader_2.54mm:PinHeader_2x09_P2.54mm_Vertical_SMD, symbol Connector_Generic:Conn_02x09_Odd_Even
- added LED19, LED20, LED21, LED22, LED23, LED24, LED25, LED26, LED27, LED28, LED29, LED30, LED31, LED32, LED33, LED34, LED35, LED36, LED37, LED38, LED39, LED40: WS2812B-2020, EnergyVortex:LED_WS2812B-B, symbol EnergyVortex:WS2812B-2020
- LED1, LED10, LED11, LED12, LED13, LED14, LED15, LED16, LED17, LED18, LED2, LED3, LED4, LED5, LED6, LED7, LED8, LED9: renamed from LED?; footprint EnergyVortex:WS2812B2020 -> EnergyVortex:LED_WS2812B-B
- S1: renamed from S25; footprint EnergyVortex:CHERRY-MX-LED -> EnergyVortex:CHERRY-MX-LED+
- S10: renamed from S2; footprint EnergyVortex:CHERRY-MX-LED -> EnergyVortex:CHERRY-MX-LED+
- S11: renamed from S3; footprint EnergyVortex:CHERRY-MX-LED -> EnergyVortex:CHERRY-MX-LED+
- S12: renamed from S4; footprint EnergyVortex:CHERRY-MX-LED -> EnergyVortex:CHERRY-MX-LED+
- S13: renamed from S5; footprint EnergyVortex:CHERRY-MX-LED -> EnergyVortex:CHERRY-MX-LED+
- S14: renamed from S6; footprint EnergyVortex:CHERRY-MX-LED -> EnergyVortex:CHERRY-MX-LED+
- S15: renamed from S7; footprint EnergyVortex:CHERRY-MX-LED -> EnergyVortex:CHERRY-MX-LED+
- S16: renamed from S8; footprint EnergyVortex:CHERRY-MX-LED -> EnergyVortex:CHERRY-MX-LED+
- S17: renamed from S9; footprint EnergyVortex:CHERRY-MX-LED -> EnergyVortex:CHERRY-MX-LED+
- S18: renamed from S10; footprint EnergyVortex:CHERRY-MX-LED -> EnergyVortex:CHERRY-MX-LED+
- S19: renamed from S11; footprint EnergyVortex:CHERRY-MX-LED -> EnergyVortex:CHERRY-MX-LED+
- S2: renamed from S26; footprint EnergyVortex:CHERRY-MX-LED -> EnergyVortex:CHERRY-MX-LED+
- S20: renamed from S12; footprint EnergyVortex:CHERRY-MX-LED -> EnergyVortex:CHERRY-MX-LED+
- S21: renamed from S13; footprint EnergyVortex:CHERRY-MX-LED -> EnergyVortex:CHERRY-MX-LED+
- S22: renamed from S14; footprint EnergyVortex:CHERRY-MX-LED -> EnergyVortex:CHERRY-MX-LED+
- S23: renamed from S15; footprint EnergyVortex:CHERRY-MX-LED -> EnergyVortex:CHERRY-MX-LED+
- S24: renamed from S16; footprint EnergyVortex:CHERRY-MX-LED -> EnergyVortex:CHERRY-MX-LED+
- S25: renamed from S17; footprint EnergyVortex:CHERRY-MX-LED -> EnergyVortex:CHERRY-MX-LED+
- S26: renamed from S18; footprint EnergyVortex:CHERRY-MX-LED -> EnergyVortex:CHERRY-MX-LED+
- S27: renamed from S19; footprint EnergyVortex:CHERRY-MX-LED -> EnergyVortex:CHERRY-MX-LED+
- S28: renamed from S20; footprint EnergyVortex:CHERRY-MX-LED -> EnergyVortex:CHERRY-MX-LED+
- S29: renamed from S21; footprint EnergyVortex:CHERRY-MX-LED -> EnergyVortex:CHERRY-MX-LED+
- S3: renamed from S27; footprint EnergyVortex:CHERRY-MX-LED -> EnergyVortex:CHERRY-MX-LED+
- S30: renamed from S22; footprint EnergyVortex:CHERRY-MX-LED -> EnergyVortex:CHERRY-MX-LED+
- S31: renamed from S23; footprint EnergyVortex:CHERRY-MX-LED -> EnergyVortex:CHERRY-MX-LED+
- S32: renamed from S24; footprint EnergyVortex:CHERRY-MX-LED -> EnergyVortex:CHERRY-MX-LED+
- S33: renamed from S35; footprint EnergyVortex:CHERRY-MX-LED -> EnergyVortex:CHERRY-MX-LED+
- S34: renamed from S36; footprint EnergyVortex:CHERRY-MX-LED -> EnergyVortex:CHERRY-MX-LED+
- S35: renamed from S37; footprint EnergyVortex:CHERRY-MX-LED -> EnergyVortex:CHERRY-MX-LED+
- S36: renamed from S38; footprint EnergyVortex:CHERRY-MX-LED -> EnergyVortex:CHERRY-MX-LED+
- S37: renamed from S39; footprint EnergyVortex:CHERRY-MX-LED -> EnergyVortex:CHERRY-MX-LED+
- S38: renamed from S40; footprint EnergyVortex:CHERRY-MX-LED -> EnergyVortex:CHERRY-MX-LED+
- S39: renamed from S33; footprint EnergyVortex:CHERRY-MX-LED -> EnergyVortex:CHERRY-MX-LED+
- S4: renamed from S28; footprint EnergyVortex:CHERRY-MX-LED -> EnergyVortex:CHERRY-MX-LED+
- S40: renamed from S34; footprint EnergyVortex:CHERRY-MX-LED -> EnergyVortex:CHERRY-MX-LED+
- S5: renamed from S29; footprint EnergyVortex:CHERRY-MX-LED -> EnergyVortex:CHERRY-MX-LED+
- S6: renamed from S30; footprint EnergyVortex:CHERRY-MX-LED -> EnergyVortex:CHERRY-MX-LED+
- S7: renamed from S31; footprint EnergyVortex:CHERRY-MX-LED -> EnergyVortex:CHERRY-MX-LED+
- S8: renamed from S32; footprint EnergyVortex:CHERRY-MX-LED -> EnergyVortex:CHERRY-MX-LED+
- S9: renamed from S1; footprint EnergyVortex:CHERRY-MX-LED -> EnergyVortex:CHERRY-MX-LED+
- SW1: renamed from SW?; footprint Button_Switch_SMD:SW_Push_1P1T_NO_6x6mm_H9.5mm -> EnergyVortex:SW_Push_1P1T_NO_6x6mm_H9.5mm
- Y1, Y2: renamed from Y?; footprint Crystal:Crystal_SMD_Qantek_QC5CB-2Pin_5x3.2mm -> EnergyVortex:Crystal_SMD_Qantek_QC5CB-2Pin_5x3.2mm
- gave numbers to parts that had none: 43
- renumbered C3 to C16, C2 to C17, C1 to C18, J1 to J7, R3 to R14, R1 to R16, R2 to R17, RN4 to RN1, RN1 to RN2, RN2 to RN3, RN3 to RN4, RN7 to RN5, RN5 to RN7, U5 to U10, U7 to U6, U6 to U7
Connections:
- net SPI1_CLK is gone; now on net SPI_1CLK: U5.21 (PA5)
- net 3.3V: now also LED19.4 (VDD), LED20.4 (VDD), LED21.4 (VDD), LED22.4 (VDD), LED23.4 (VDD), LED24.4 (VDD), LED25.4 (VDD), LED26.4 (VDD), LED27.4 (VDD), LED28.4 (VDD), LED29.4 (VDD), LED30.4 (VDD), LED31.4 (VDD), LED32.4 (VDD), LED33.4 (VDD), LED34.4 (VDD), LED35.4 (VDD), LED36.4 (VDD), LED37.4 (VDD), LED38.4 (VDD), LED39.4 (VDD), LED40.4 (VDD)
- net 5V: now also JP1.2 (B), JP2.2 (B)
- net GND: now also LED12.2 (GND), LED18.2 (GND), LED3.2 (GND), LED9.2 (GND), LED19.2 (GND), LED20.2 (GND), LED21.2 (GND), LED22.2 (GND), LED23.2 (GND), LED24.2 (GND), LED25.2 (GND), LED26.2 (GND), LED27.2 (GND), LED28.2 (GND), LED29.2 (GND), LED30.2 (GND), LED31.2 (GND), LED32.2 (GND), LED33.2 (GND), LED34.2 (GND), LED35.2 (GND), LED36.2 (GND), LED37.2 (GND), LED38.2 (GND), LED39.2 (GND), LED40.2 (GND)
- net PA15: now also J2.6 (Pin_6)
- net PA2: now also J2.1 (Pin_1)
- net PA3: now also J2.2 (Pin_2)
- net PA4: now also J2.3 (Pin_3)
- net PA7: now also J2.4 (Pin_4)
- net PA8: now also J2.5 (Pin_5)
- net PB0: now also J2.7 (Pin_7)
- net PB1: now also J2.8 (Pin_8)
- net PB10: now also J2.16 (Pin_16)
- net PB11: now also J2.17 (Pin_17)
- net PB12: now also J2.18 (Pin_18)
- net PB14: now also J3.1 (Pin_1)
- net PB3: now also J2.9 (Pin_9)
- net PB4: now also J2.10 (Pin_10)
- net PB5: now also J2.11 (Pin_11)
- net PB6: now also J2.12 (Pin_12)
- net PB7: now also J2.13 (Pin_13)
- net PB8: now also J2.14 (Pin_14)
- net PB9: now also J2.15 (Pin_15)
- net PC0: now also J3.2 (Pin_2)
- net PC1: now also J3.3 (Pin_3)
- net PC10: now also J3.12 (Pin_12)
- net PC11: now also J3.13 (Pin_13)
- net PC12: now also J3.14 (Pin_14)
- net PC13: now also J3.15 (Pin_15)
- net PC14: now also J3.16 (Pin_16)
- net PC15: now also J3.17 (Pin_17)
- net PC2: now also J3.4 (Pin_4)
- net PC3: now also J3.5 (Pin_5)
- net PC4: now also J3.6 (Pin_6)
- net PC5: now also J3.7 (Pin_7)
- net PC6: now also J3.8 (Pin_8)
- net PC7: now also J3.9 (Pin_9)
- net PC8: now also J3.10 (Pin_10)
- net PC9: now also J3.11 (Pin_11)
- net PD2: now also J3.18 (Pin_18)
- net SCAN_PL: no longer U1.9 (QH)
- net SPI_KEY2: now also LED19.3 (DI)
- net SPI1_MISO renamed SPI_1MISO
- net SPI_1MISO: now also U1.9 (QH)
- new net: LED39.1 (DO), LED40.3 (DI)
- new net: LED38.1 (DO), LED39.3 (DI)
- new net: LED35.1 (DO), LED36.3 (DI)
- new net: LED31.1 (DO), LED32.3 (DI)
- new net: LED30.1 (DO), LED31.3 (DI)
- new net: LED28.1 (DO), LED29.3 (DI)
- new net: LED33.1 (DO), LED34.3 (DI)
- new net: LED32.1 (DO), LED33.3 (DI)
- new net: LED23.1 (DO), LED24.3 (DI)
- new net: LED22.1 (DO), LED23.3 (DI)
- new net: LED24.1 (DO), LED25.3 (DI)
- new net: LED21.1 (DO), LED22.3 (DI)
- new net: LED26.1 (DO), LED27.3 (DI)
- new net: LED25.1 (DO), LED26.3 (DI)
- new net: LED19.1 (DO), LED20.3 (DI)
- new net: LED20.1 (DO), LED21.3 (DI)
- new net: LED34.1 (DO), LED35.3 (DI)
- new net: LED29.1 (DO), LED30.3 (DI)
- new net: LED37.1 (DO), LED38.3 (DI)
- new net SPI_KEY3: LED27.1 (DO), LED28.3 (DI)
- new net SPI_KEY4: LED36.1 (DO), LED37.3 (DI)
Other:
- note added: "5V to 3.3V"
- note added: "BOOT控制器"
- note added: "ST-LINK下载口"
- note added: "USB"
- note added: "USB转UART,CH340"
- note added: "串口调试口"
- moved on the sheet: C12, C14, D1, D3, J1, J4, J6, JP1, JP2, LED1, LED10, LED11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
